File: CRUCE POR CERO/CRUCE POR CERO.kicad_pcb (KiCad board)
At the start: 2 copper layers, 50.4 x 41.1 mm, 17 parts, among them J1 F, J2 CRUCE POR CERO, J3 N, J4 CONTROL, J5 SSR+CALEFACTOR, U1 H11AA1

Commit message: actualización
Parts:
- removed RV1: 14D471K 470Vpp, Varistor:RV_Disc_D15.5mm_W7.5mm_P7.5mm
- J1, J3: footprint Connector_PinHeader_2.00mm:PinHeader_1x01_P2.00mm_Vertical -> Connector_PinSocket_2.54mm:PinSocket_1x01_P2.54mm_Vertical
- J4: value CONTROL -> 220V para FUENTE 5V
- J5: value SSR+CALEFACTOR -> SSR y CALEFACTOR
- moved R1 1.30 mm to (113.0, 98.7), turned to -90 degrees
- moved C1 0.51 mm to (116.4, 103.7), turned to 90 degrees
- moved J2 0.38 mm to (116.4, 107.6)
Routing:
- net F: track 243.5 -> 27.5 mm
- net N: track 215.4 -> 48.9 mm
- net Net-(J2-Pin_2): track 13.7 -> 25.3 mm
- net Net-(J2-Pin_1): track 15.4 -> 19.6 mm
- added copper zone on B.Cu, net F
- added copper zone on B.Cu, net N

Commit message: Add files via upload
Parts:
- F1: value 220V 7A -> 230V 7A
- J4: value 220V para FUENTE 5V -> 230V para FUENTE 5V
Changed lines of the file:
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@@
 			)
 		)
-		(property "Value" "220V 7A"
+		(property "Value" "230V 7A"
 			(at -5.75 -5.93 0)
 			(layer "F.Fab")
@@
 			)
 		)
-		(property "Value" "220V para FUENTE 5V"
+		(property "Value" "230V para FUENTE 5V"
 			(at -0.83 5.25 0)
 			(layer "F.Fab")
