File: CRUCE POR CERO/CRUCE POR CERO.kicad_sch (KiCad schematic)
At the start: 17 parts, among them J1 F, J2 CRUCE POR CERO, J3 N, J4 CONTROL, J5 SSR+CALEFACTOR, U1 H11AA1

Commit message: actualización
Parts:
- J1, J3: footprint Connector_PinHeader_2.00mm:PinHeader_1x01_P2.00mm_Vertical -> Connector_PinSocket_2.54mm:PinSocket_1x01_P2.54mm_Vertical
- J4: value CONTROL -> 220V PARA PCB DE CONTROL
- J5: value SSR+CALEFACTOR -> SSR / CALEFACTOR
Other:
- moved on the sheet: C1, H1, H2, H3, H4, J4, J5, R2, R3, R4

Commit message: Add files via upload
Other:
- note added: "DETECCION DE CRUCE POR CERO (230V)"
- note removed: "DETECCION DE CRUCE POR CERO (220V)"
Changed lines of the file:
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@@
 	(generator_version "9.0")
 	(paper "A4")
-	(text "DETECCION DE CRUCE POR CERO (220V)\n"
+	(text "DETECCION DE CRUCE POR CERO (230V)\n"
 		(exclude_from_sim no)
 		(at 96.52 74.676 0)
